File: kicad/superhashtagpcb.kicad_pcb (KiCad board)
At the start: 2 copper layers, 99 x 79.6 mm, 3 parts

Commit message: adding schema and layout position changes.
Parts:
- removed G*** (x3): LOGO, LOGO
- added ? (x2): , LOGO, F.Cu at (150.0, 115.0)

Commit message: initial layout, pre coper
Parts:
- removed the ? at (150.0, 115.0) (x2)
- added ?: , superhashtagpcb:B.Mask_g8161, F.Cu at (150.0, 115.0)
- added ?: , superhashtagpcb:B.Silk_g8163, F.Cu at (150.0, 115.0)
- added BT1: Battery, Battery:BatteryHolder_Keystone_3034_1x20mm, F.Cu at (149.9, 132.1)
- added D1: LED, DigiKey:LED_5mm_Radial, B.Cu at (116.8, 85.1)
- added D2: LED, DigiKey:LED_5mm_Radial, B.Cu at (110.5, 94.0)
- added R1: R, Resistor_THT:R_Axial_DIN0207_L6.3mm_D2.5mm_P10.16mm_Horizontal, F.Cu at (129.5, 100.3)
- added R2: R, Resistor_THT:R_Axial_DIN0207_L6.3mm_D2.5mm_P10.16mm_Horizontal, F.Cu at (129.5, 96.5)
- added SW1: SW_DPDT_x2, DigiKey:Switch_Toggle_ATE1D-2M3-10-Z, F.Cu at (116.8, 108.0)

Commit message: placed traces and vias
Parts:
- moved R1 3.81 mm to (129.5, 96.5)
- moved R2 2.54 mm to (129.5, 99.1)
Routing:
- net GND: track 0.00 -> 25.5 mm, vias 0 -> 1
- net Net-(R1-Pad1): track 0.00 -> 18.9 mm
- net Net-(D1-Pad2): track 0.00 -> 13.4 mm
- net Net-(D2-Pad2): track 0.00 -> 11.0 mm
- added copper zone on F.Cu, net /VCC
- added copper zone on B.Cu, net GND
