File: 04-H+H_sao/04-H+H_sao.sch (KiCad schematic (older format))
At the start: 8 parts, among them U1 ICM7555, X1 Badgelife_sao_connector_v169b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

Commit message: rerouted sao
Parts:
- U1: footprint Package_DIP:DIP-8_W7.62mm_SMDSocket_SmallPads -> ICM7555IBAZ-T:SOIC127P600X175-8N
Changed lines of the file:
@@
 F 0 "U1" H 5100 4028 50  0000 C CNN
 F 1 "ICM7555" H 5100 3937 50  0000 C CNN
-F 2 "Package_DIP:DIP-8_W7.62mm_SMDSocket_SmallPads" H 5100 3450 50  0001 C CNN
+F 2 "ICM7555IBAZ-T:SOIC127P600X175-8N" H 5100 3450 50  0001 C CNN
 F 3 "http://www.intersil.com/content/dam/Intersil/documents/icm7/icm7555-56.pdf" H 5100 3450 50  0001 C CNN
 	1    5100 3450
